File: breakout.sch (KiCad schematic (older format))
At the start: 11 parts, among them P1 CONN_01X09, P2 CONN_01X09, U1 ESP-12E, U2 HT7333

Commit message: Switch back to the SPX regulator.
Parts:
- removed U2: HT7333, TO_SOT_Packages_SMD:SOT89-3_Housing_Handsoldering, symbol APE8865N-33-HF-3
- added U2: SPX3819M5-L-3-3, TO_SOT_Packages_SMD:SOT-23-5, symbol APE8865Y5-33-HF-3
Connections:
- net +12V: now also U2.1 (VIN), U2.3 (~SHDN~)
- net 3V3: now also U2.5 (VOUT)
- net GND: now also U2.2 (GND)
- no-connect marks 6 -> 7
Changed lines of the file:
@@
 	1    0    0    -1
 $EndComp
-Wire Wire Line
-	3800 2950 4700 2950
-Wire Wire Line
-	4700 3050 3800 3050
-Wire Wire Line
-	3800 3150 4700 3150
-Wire Wire Line
-	4700 3250 3800 3250
-Wire Wire Line
-	3800 3350 4700 3350
-Wire Wire Line
-	4700 3450 3800 3450
-Wire Wire Line
-	3800 3550 4700 3550
-Wire Wire Line
-	6500 2950 7000 2950
-Wire Wire Line
-	6500 3050 7000 3050
-Wire Wire Line
-	7000 3150 6500 3150
-Wire Wire Line
-	6500 3250 7000 3250
-Wire Wire Line
-	6500 3350 7000 3350
-Wire Wire Line
-	6500 3450 7000 3450
-Wire Wire Line
-	6500 3550 7000 3550
-Wire Wire Line
-	6500 3650 7000 3650
-Wire Wire Line
-	3600 2150 6900 2150
-Wire Wire Line
-	3150 2500 3750 2500
-Wire Wire Line
-	3150 2500 3150 4250
-Wire Wire Line
-	3150 4250 6800 4250
-Wire Wire Line
-	4250 2650 4250 3150
-Connection ~ 4250 3150
-Wire Wire Line
-	4600 2650 4600 2950
-Connection ~ 4600 2950
-Wire Wire Line
-	4250 2350 4250 2150
-Connection ~ 4250 2150
-Wire Wire Line
-	4600 2150 4600 2350
-Connection ~ 4600 2150
-Wire Wire Line
-	6550 4250 6550 3650
-Connection ~ 6550 3650
-Wire Wire Line
-	6800 3550 6800 3750
-Connection ~ 6800 3550
-Wire Wire Line
-	6800 4250 6800 4050
-Connection ~ 6550 4250
-Wire Wire Line
-	4700 3650 4100 3650
-Wire Wire Line
-	4100 3650 4100 2150
-Connection ~ 4100 2150
-Wire Wire Line
-	2500 3850 3900 3850
-Wire Wire Line
-	2500 3850 2500 2150
-Wire Wire Line
-	2500 2150 2700 2150
-$Comp
-L +12V #PWR3
+$Comp
+L +12V #PWR01
 U 1 1 56841BDC
 P 2500 2150
-F 0 "#PWR3" H 2500 2000 50  0001 C CNN
+F 0 "#PWR01" H 2500 2000 50  0001 C CNN
 F 1 "+12V" V 2518 2277 50  0000 L CNN
 F 2 "" H 2500 2150 50  0000 C CNN
@@
 $EndComp
 $Comp
-L GND #PWR4
+L GND #PWR02
 U 1 1 56841C6C
 P 6800 4250
-F 0 "#PWR4" H 6800 4000 50  0001 C CNN
+F 0 "#PWR02" H 6800 4000 50  0001 C CNN
 F 1 "GND" H 6808 4076 50  0000 C CNN
 F 2 "" H 6800 4250 50  0000 C CNN
@@
 $EndComp
 $Comp
-L PWR_FLAG #FLG1
+L PWR_FLAG #FLG03
 U 1 1 56841CB3
 P 1200 2200
-F 0 "#FLG1" H 1200 2295 50  0001 C CNN
+F 0 "#FLG03" H 1200 2295 50  0001 C CNN
 F 1 "PWR_FLAG" H 1200 2423 50  0000 C CNN
 F 2 "" H 1200 2200 50  0000 C CNN
@@
 $EndComp
 $Comp
-L PWR_FLAG #FLG2
+L PWR_FLAG #FLG04
 U 1 1 56841D0E
 P 1650 2050
-F 0 "#FLG2" H 1650 2145 50  0001 C CNN
+F 0 "#FLG04" H 1650 2145 50  0001 C CNN
 F 1 "PWR_FLAG" H 1650 2274 50  0000 C CNN
 F 2 "" H 1650 2050 50  0000 C CNN
@@
 $EndComp
 $Comp
-L +12V #PWR1
+L +12V #PWR05
 U 1 1 56841D46
 P 1200 2000
-F 0 "#PWR1" H 1200 1850 50  0001 C CNN
+F 0 "#PWR05" H 1200 1850 50  0001 C CNN
 F 1 "+12V" H 1218 2174 50  0000 C CNN
 F 2 "" H 1200 2000 50  0000 C CNN
@@
 	1    0    0    -1
 $EndComp
-Wire Wire Line
-	1200 2000 1200 2200
-$Comp
-L GND #PWR2
+$Comp
+L GND #PWR06
 U 1 1 56841DA6
 P 1650 2250
-F 0 "#PWR2" H 1650 2000 50  0001 C CNN
+F 0 "#PWR06" H 1650 2000 50  0001 C CNN
 F 1 "GND" H 1658 2076 50  0000 C CNN
 F 2 "" H 1650 2250 50  0000 C CNN
@@
 	1    0    0    -1
 $EndComp
-Wire Wire Line
-	1650 2050 1650 2250
 Text Label 5100 2150 0    60   ~ 0
 3V3
@@
 	1    0    0    -1
 $EndComp
-Wire Wire Line
-	6900 2150 6900 2350
-Wire Wire Line
-	6550 2350 6550 2150
-Connection ~ 6550 2150
-Wire Wire Line
-	6550 2650 6550 3350
-Connection ~ 6550 3350
-Wire Wire Line
-	6900 2650 6900 3450
-Connection ~ 6900 3450
 $Comp
 L CONN_01X09 P1
@@
 	-1   0    0    -1
 $EndComp
-Wire Wire Line
-	3900 3850 3900 3650
-Wire Wire Line
-	3900 3650 3800 3650
-Wire Wire Line
-	3800 3750 4200 3750
-Wire Wire Line
-	4200 3750 4200 3650
-Connection ~ 4200 3650
-Wire Wire Line
-	3750 2200 3750 2150
-Connection ~ 3750 2150
 $Comp
 L CONN_01X09 P2
@@
 	1    0    0    -1
 $EndComp
-Wire Wire Line
-	6900 3650 6900 3750
-Wire Wire Line
-	6900 3750 7000 3750
-Connection ~ 6900 3650
 $Comp
 L C C2
@@
 	0    1    1    0
 $EndComp
+$Comp
+L APE8865Y5-33-HF-3 U2
+U 1 1 5696F404
+P 3150 2200
+F 0 "U2" H 2850 2500 50  0000 C CNN
+F 1 "SPX3819M5-L-3-3" H 3150 2400 50  0000 C CNN
+F 2 "TO_SOT_Packages_SMD:SOT-23-5" H 3150 2300 50  0000 C CIN
+F 3 "" H 3150 2200 50  0000 C CNN
+	1    3150 2200
+	1    0    0    -1
+$EndComp
+Wire Wire Line
+	3800 2950 4700 2950
+Wire Wire Line
+	4700 3050 3800 3050
+Wire Wire Line
+	3800 3150 4700 3150
+Wire Wire Line
+	4700 3250 3800 3250
+Wire Wire Line
+	3800 3350 4700 3350
+Wire Wire Line
+	4700 3450 3800 3450
+Wire Wire Line
+	3800 3550 4700 3550
+Wire Wire Line
+	6500 2950 7000 2950
+Wire Wire Line
+	6500 3050 7000 3050
+Wire Wire Line
+	7000 3150 6500 3150
+Wire Wire Line
+	6500 3250 7000 3250
+Wire Wire Line
+	6500 3350 7000 3350
+Wire Wire Line
+	6500 3450 7000 3450
+Wire Wire Line
+	6500 3550 7000 3550
+Wire Wire Line
+	6500 3650 7000 3650
+Wire Wire Line
+	3600 2150 6900 2150
+Wire Wire Line
+	3150 2500 3750 2500
+Wire Wire Line
+	3150 2500 3150 4250
+Wire Wire Line
+	3150 4250 6800 4250
+Wire Wire Line
+	4250 2650 4250 3150
+Connection ~ 4250 3150
+Wire Wire Line
+	4600 2650 4600 2950
+Connection ~ 4600 2950
+Wire Wire Line
+	4250 2350 4250 2150
+Connection ~ 4250 2150
+Wire Wire Line
+	4600 2150 4600 2350
+Connection ~ 4600 2150
+Wire Wire Line
+	6550 4250 6550 3650
+Connection ~ 6550 3650
+Wire Wire Line
+	6800 3550 6800 3750
+Connection ~ 6800 3550
+Wire Wire Line
+	6800 4250 6800 4050
+Connection ~ 6550 4250
+Wire Wire Line
+	4700 3650 4100 3650
+Wire Wire Line
+	4100 3650 4100 2150
+Connection ~ 4100 2150
+Wire Wire Line
+	2500 3850 3900 3850
+Wire Wire Line
+	2500 3850 2500 2150
+Wire Wire Line
+	2500 2150 2700 2150
+Wire Wire Line
+	1200 2000 1200 2200
+Wire Wire Line
+	1650 2050 1650 2250
+Wire Wire Line
+	6900 2150 6900 2350
+Wire Wire Line
+	6550 2350 6550 2150
+Connection ~ 6550 2150
+Wire Wire Line
+	6550 2650 6550 3350
+Connection ~ 6550 3350
+Wire Wire Line
+	6900 2650 6900 3450
+Connection ~ 6900 3450
+Wire Wire Line
+	3900 3850 3900 3650
+Wire Wire Line
+	3900 3650 3800 3650
+Wire Wire Line
+	3800 3750 4200 3750
+Wire Wire Line
+	4200 3750 4200 3650
+Connection ~ 4200 3650
+Wire Wire Line
+	3750 2200 3750 2150
+Connection ~ 3750 2150
+Wire Wire Line
+	6900 3650 6900 3750
+Wire Wire Line
+	6900 3750 7000 3750
+Connection ~ 6900 3650
 Wire Wire Line
 	2650 2650 2500 2650
@@
 	2950 2650 3150 2650
 Connection ~ 3150 2650
-$Comp
-L APE8865N-33-HF-3 U2
-U 1 1 5694FDB4
-P 3150 2200
-F 0 "U2" H 3150 2500 50  0000 C CNN
-F 1 "HT7333" H 3150 2400 50  0000 C CNN
-F 2 "TO_SOT_Packages_SMD:SOT89-3_Housing_Handsoldering" H 3150 2300 50  0001 C CIN
-F 3 "" H 3150 2200 50  0000 C CNN
-	1    3150 2200
-	1    0    0    -1
-$EndComp
+Wire Wire Line
+	2700 2300 2650 2300
+Wire Wire Line
+	2650 2300 2650 2150
+Connection ~ 2650 2150
+NoConn ~ 3600 2300
 $EndSCHEMATC

Commit message: Make PCB a bit smaller.
Parts:
- added P3: USB_OTG, Connect:USB_Micro-B_10103594-0001LF, symbol USB_OTG
Connections:
- net GND: now also P3.5 (GND)
- net +12V renamed +5V
- net +5V: now also P3.1 (VCC)
Changed lines of the file:
@@
 $EndComp
 $Comp
-L +12V #PWR01
-U 1 1 56841BDC
-P 2500 2150
-F 0 "#PWR01" H 2500 2000 50  0001 C CNN
-F 1 "+12V" V 2518 2277 50  0000 L CNN
-F 2 "" H 2500 2150 50  0000 C CNN
-F 3 "" H 2500 2150 50  0000 C CNN
-	1    2500 2150
-	0    -1   -1   0
-$EndComp
-$Comp
-L GND #PWR02
+L GND #PWR01
 U 1 1 56841C6C
 P 6800 4250
-F 0 "#PWR02" H 6800 4000 50  0001 C CNN
+F 0 "#PWR01" H 6800 4000 50  0001 C CNN
 F 1 "GND" H 6808 4076 50  0000 C CNN
 F 2 "" H 6800 4250 50  0000 C CNN
@@
 $EndComp
 $Comp
-L PWR_FLAG #FLG03
+L PWR_FLAG #FLG02
 U 1 1 56841CB3
 P 1200 2200
-F 0 "#FLG03" H 1200 2295 50  0001 C CNN
+F 0 "#FLG02" H 1200 2295 50  0001 C CNN
 F 1 "PWR_FLAG" H 1200 2423 50  0000 C CNN
 F 2 "" H 1200 2200 50  0000 C CNN
@@
 $EndComp
 $Comp
-L PWR_FLAG #FLG04
+L PWR_FLAG #FLG03
 U 1 1 56841D0E
 P 1650 2050
-F 0 "#FLG04" H 1650 2145 50  0001 C CNN
+F 0 "#FLG03" H 1650 2145 50  0001 C CNN
 F 1 "PWR_FLAG" H 1650 2274 50  0000 C CNN
 F 2 "" H 1650 2050 50  0000 C CNN
@@
 $EndComp
 $Comp
-L +12V #PWR05
-U 1 1 56841D46
-P 1200 2000
-F 0 "#PWR05" H 1200 1850 50  0001 C CNN
-F 1 "+12V" H 1218 2174 50  0000 C CNN
-F 2 "" H 1200 2000 50  0000 C CNN
-F 3 "" H 1200 2000 50  0000 C CNN
-	1    1200 2000
-	1    0    0    -1
-$EndComp
-$Comp
-L GND #PWR06
+L GND #PWR04
 U 1 1 56841DA6
 P 1650 2250
-F 0 "#PWR06" H 1650 2000 50  0001 C CNN
+F 0 "#PWR04" H 1650 2000 50  0001 C CNN
 F 1 "GND" H 1658 2076 50  0000 C CNN
 F 2 "" H 1650 2250 50  0000 C CNN
@@
 F 0 "U2" H 2850 2500 50  0000 C CNN
 F 1 "SPX3819M5-L-3-3" H 3150 2400 50  0000 C CNN
-F 2 "TO_SOT_Packages_SMD:SOT-23-5" H 3150 2300 50  0000 C CIN
+F 2 "TO_SOT_Packages_SMD:SOT-23-5" H 3150 2300 50  0001 C CIN
 F 3 "" H 3150 2200 50  0000 C CNN
 	1    3150 2200
@@
 Connection ~ 6550 4250
 Wire Wire Line
-	4700 3650 4100 3650
+	4100 3650 4700 3650
 Wire Wire Line
 	4100 3650 4100 2150
@@
 	2500 3850 3900 3850
 Wire Wire Line
-	2500 3850 2500 2150
+	2500 1550 2500 3850
 Wire Wire Line
 	2500 2150 2700 2150
@@
 Connection ~ 2650 2150
 NoConn ~ 3600 2300
+$Comp
+L USB_OTG P3
+U 1 1 56AB8797
+P 3150 1300
+F 0 "P3" H 3475 1175 50  0000 C CNN
+F 1 "USB_OTG" H 3150 1500 50  0000 C CNN
+F 2 "Connect:USB_Micro-B_10103594-0001LF" V 3100 1200 50  0001 C CNN
+F 3 "" V 3100 1200 50  0000 C CNN
+	1    3150 1300
+	1    0    0    -1
+$EndComp
+Wire Wire Line
+	2950 1600 2500 1600
+Connection ~ 2500 2150
+$Comp
+L GND #PWR05
+U 1 1 56AB8ABD
+P 3350 1650
+F 0 "#PWR05" H 3350 1400 50  0001 C CNN
+F 1 "GND" H 3358 1476 50  0000 C CNN
+F 2 "" H 3350 1650 50  0000 C CNN
+F 3 "" H 3350 1650 50  0000 C CNN
+	1    3350 1650
+	1    0    0    -1
+$EndComp
+Wire Wire Line
+	3350 1600 3350 1650
+$Comp
+L +5V #PWR06
+U 1 1 56AB8C2F
+P 1200 2000
+F 0 "#PWR06" H 1200 1850 50  0001 C CNN
+F 1 "+5V" H 1200 2140 50  0000 C CNN
+F 2 "" H 1200 2000 50  0000 C CNN
+F 3 "" H 1200 2000 50  0000 C CNN
+	1    1200 2000
+	1    0    0    -1
+$EndComp
+$Comp
+L +5V #PWR07
+U 1 1 56AB8C65
+P 2500 1550
+F 0 "#PWR07" H 2500 1400 50  0001 C CNN
+F 1 "+5V" H 2500 1690 50  0000 C CNN
+F 2 "" H 2500 1550 50  0000 C CNN
+F 3 "" H 2500 1550 50  0000 C CNN
+	1    2500 1550
+	1    0    0    -1
+$EndComp
+Connection ~ 2500 1600
 $EndSCHEMATC

Commit message: Remove erroneous USB_OTG component.
Parts:
- removed P3: USB_OTG, Connect:USB_Micro-B_10103594-0001LF, symbol USB_OTG
Changed lines of the file:
@@
 	2500 3850 3900 3850
 Wire Wire Line
-	2500 1550 2500 3850
+	2500 2000 2500 3850
 Wire Wire Line
 	2500 2150 2700 2150
@@
 Connection ~ 2650 2150
 NoConn ~ 3600 2300
-$Comp
-L USB_OTG P3
-U 1 1 56AB8797
-P 3150 1300
-F 0 "P3" H 3475 1175 50  0000 C CNN
-F 1 "USB_OTG" H 3150 1500 50  0000 C CNN
-F 2 "Connect:USB_Micro-B_10103594-0001LF" V 3100 1200 50  0001 C CNN
-F 3 "" V 3100 1200 50  0000 C CNN
-	1    3150 1300
-	1    0    0    -1
-$EndComp
-Wire Wire Line
-	2950 1600 2500 1600
 Connection ~ 2500 2150
 $Comp
-L GND #PWR05
-U 1 1 56AB8ABD
-P 3350 1650
-F 0 "#PWR05" H 3350 1400 50  0001 C CNN
-F 1 "GND" H 3358 1476 50  0000 C CNN
-F 2 "" H 3350 1650 50  0000 C CNN
-F 3 "" H 3350 1650 50  0000 C CNN
-	1    3350 1650
-	1    0    0    -1
-$EndComp
-Wire Wire Line
-	3350 1600 3350 1650
-$Comp
-L +5V #PWR06
+L +5V #PWR05
 U 1 1 56AB8C2F
 P 1200 2000
-F 0 "#PWR06" H 1200 1850 50  0001 C CNN
+F 0 "#PWR05" H 1200 1850 50  0001 C CNN
 F 1 "+5V" H 1200 2140 50  0000 C CNN
 F 2 "" H 1200 2000 50  0000 C CNN
@@
 $EndComp
 $Comp
-L +5V #PWR07
+L +5V #PWR06
 U 1 1 56AB8C65
-P 2500 1550
-F 0 "#PWR07" H 2500 1400 50  0001 C CNN
-F 1 "+5V" H 2500 1690 50  0000 C CNN
-F 2 "" H 2500 1550 50  0000 C CNN
-F 3 "" H 2500 1550 50  0000 C CNN
-	1    2500 1550
+P 2500 2000
+F 0 "#PWR06" H 2500 1850 50  0001 C CNN
+F 1 "+5V" H 2500 2140 50  0000 C CNN
+F 2 "" H 2500 2000 50  0000 C CNN
+F 3 "" H 2500 2000 50  0000 C CNN
+	1    2500 2000
 	1    0    0    -1
 $EndComp
-Connection ~ 2500 1600
 $EndSCHEMATC
