File: breakout.sch (KiCad schematic (older format))
At the start: 11 parts, among them P1 CONN_01X09, P2 CONN_01X09, U1 ESP-12E, U2 SPX3819M5-L-3-3

Commit message: Change caps to 22uF.
Parts:
- C1, C2: value 10uF -> 22uF
Changed lines of the file:
@@
 P 3750 2350
 F 0 "C1" H 3865 2442 50  0000 L CNN
-F 1 "10uF" H 3865 2350 50  0000 L CNN
+F 1 "22uF" H 3865 2350 50  0000 L CNN
 F 2 "Capacitors_SMD:C_0805_HandSoldering" H 3865 2258 50  0001 L CNN
 F 3 "" H 3750 2350 50  0000 C CNN
@@
 P 2800 2650
 F 0 "C2" H 2915 2742 50  0000 L CNN
-F 1 "10uF" H 2915 2650 50  0000 L CNN
+F 1 "22uF" H 2915 2650 50  0000 L CNN
 F 2 "Capacitors_SMD:C_0805_HandSoldering" H 2915 2558 50  0001 L CNN
 F 3 "" H 2800 2650 50  0000 C CNN

Commit message: Make an even tinier PCB
Parts:
- removed P1, P2: CONN_01X09, Pin_Headers:Pin_Header_Straight_1x09, symbol CONN_01X09
- added J1: Conn_01x01, Pin_Headers:Pin_Header_Straight_1x01_Pitch1.00mm, symbol Conn_01x01
- U2: symbol APE8865Y5-33-HF-3 -> APE8865Y5-33-HF-3-RESCUE-breakout
Connections:
- net +5V: now also J1.1 (Pin_1)
- no-connect marks 7 -> 25
Changed lines of the file:
@@
 EESchema Schematic File Version 2
+LIBS:breakout-rescue
 LIBS:power
 LIBS:device
@@
 $EndComp
 $Comp
-L CONN_01X09 P1
-U 1 1 568C725D
-P 3600 3350
-F 0 "P1" H 3600 3850 50  0000 C CNN
-F 1 "CONN_01X09" V 3700 3350 50  0000 C CNN
-F 2 "Pin_Headers:Pin_Header_Straight_1x09" H 3600 3350 50  0001 C CNN
-F 3 "" H 3600 3350 50  0000 C CNN
-	1    3600 3350
-	-1   0    0    -1
-$EndComp
-$Comp
-L CONN_01X09 P2
-U 1 1 568C7A2E
-P 7200 3350
-F 0 "P2" H 7200 3850 50  0000 C CNN
-F 1 "CONN_01X09" V 7300 3350 50  0000 C CNN
-F 2 "Pin_Headers:Pin_Header_Straight_1x09" H 7200 3350 50  0001 C CNN
-F 3 "" H 7200 3350 50  0000 C CNN
-	1    7200 3350
-	1    0    0    -1
-$EndComp
-$Comp
 L C C2
 U 1 1 5694F907
@@
 $EndComp
 $Comp
-L APE8865Y5-33-HF-3 U2
+L APE8865Y5-33-HF-3-RESCUE-breakout U2
 U 1 1 5696F404
 P 3150 2200
@@
 	1    0    0    -1
 $EndComp
+NoConn ~ 3800 3750
+NoConn ~ 3800 3650
+NoConn ~ 3800 3550
+NoConn ~ 3800 3450
+NoConn ~ 3800 3350
+NoConn ~ 3800 3250
+NoConn ~ 3800 3150
+NoConn ~ 3800 3050
+NoConn ~ 3800 2950
+NoConn ~ 7000 2950
+NoConn ~ 7000 3050
+NoConn ~ 7000 3150
+NoConn ~ 7000 3250
+NoConn ~ 7000 3350
+NoConn ~ 7000 3450
+NoConn ~ 7000 3550
+NoConn ~ 7000 3650
+NoConn ~ 7000 3750
+$Comp
+L Conn_01x01 J1
+U 1 1 5BA3118D
+P 2150 2800
+F 0 "J1" H 2150 2900 50  0000 C CNN
+F 1 "Conn_01x01" H 2150 2700 50  0000 C CNN
+F 2 "Pin_Headers:Pin_Header_Straight_1x01_Pitch1.00mm" H 2150 2800 50  0001 C CNN
+F 3 "" H 2150 2800 50  0001 C CNN
+	1    2150 2800
+	-1   0    0    1
+$EndComp
+Wire Wire Line
+	2350 2800 2500 2800
+Connection ~ 2500 2800
 $EndSCHEMATC
